File: ornament2023/ornament2023.kicad_sch (KiCad schematic)
At the start: 18 parts, among them J1 Conn_01x03, SW1 SW_Push, SW2 SW_DPDT_x2, U1 ATtiny404-SS

Commit message: kinda just sat down and did this all in one go
Other:
- note added: "No longer dependent on PB2, and so PWM on all pins exists now?"
- note removed: "No longer dependent on PB2, and so PWN on all pins exists now"
Changed lines of the file:
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@@
     (stroke (width 0) (type default) (color 0 0 0 0))
   )
-  (text "No longer dependent on PB2,\nand so PWN on all pins exists\nnow"
+  (text "No longer dependent on PB2,\nand so PWM on all pins exists\nnow?"
     (at 39.37 62.23 0)
     (effects (font (size 1.27 1.27)) (justify left bottom))
